File: pcb/RishiStarbie.kicad_pcb (KiCad board)
At the start: 2 copper layers, 94.7 x 90.4 mm, 7 parts, among them J1 OLED, J2 MPU6050, SW1 MX switch, SW2 MX switch, U1 XIAO-ESP32-C3, U2 DHT11

Commit message: Move off-board XIAO silkscreen to fab layer, rename footprint to XIAO-ESP32-C3-DIP
Parts:
- U1: footprint Imported Parts:XIAO-ESP32-C6-DIP -> Imported Parts:XIAO-ESP32-C3-DIP
Changed lines of the file:
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@@
     )
   )
-  (footprint "Imported Parts:XIAO-ESP32-C6-DIP" (layer "F.Cu")
+  (footprint "Imported Parts:XIAO-ESP32-C3-DIP" (layer "F.Cu")
     (at 119.5 124.9815 -90)
     (attr smd)
@@
     (fp_line (start -10.414 -6.985) (end -10.414 6.985)
       (stroke (width 0.127) (type solid)) (layer "F.SilkS"))
-    (fp_line (start -8.509 -8.89) (end 8.636 -8.89)
-      (stroke (width 0.127) (type solid)) (layer "F.SilkS"))
-    (fp_line (start -8.509 8.89) (end 8.636 8.89)
-      (stroke (width 0.127) (type solid)) (layer "F.SilkS"))
-    (fp_line (start 10.541 -4.495) (end 11.551272 -4.491272)
-      (stroke (width 0.127) (type solid)) (layer "F.SilkS"))
-    (fp_line (start 10.541 6.985) (end 10.541 -6.985)
-      (stroke (width 0.1) (type solid)) (layer "F.SilkS"))
-    (fp_line (start 10.541 6.985) (end 10.541 -6.985)
-      (stroke (width 0.127) (type solid)) (layer "F.SilkS"))
-    (fp_line (start 11.551 4.504) (end 10.541 4.504)
-      (stroke (width 0.127) (type solid)) (layer "F.SilkS"))
-    (fp_line (start 12.051 -3.991272) (end 12.051 4.004)
-      (stroke (width 0.127) (type solid)) (layer "F.SilkS"))
     (fp_arc (start -10.414 -6.985) (mid -9.856038 -8.332038) (end -8.509 -8.89)
       (stroke (width 0.127) (type solid)) (layer "F.SilkS"))
     (fp_arc (start -8.509 8.89) (mid -9.856038 8.332038) (end -10.414 6.985)
       (stroke (width 0.127) (type solid)) (layer "F.SilkS"))
-    (fp_arc (start 8.636 -8.89) (mid 9.983038 -8.332038) (end 10.541 -6.985)
-      (stroke (width 0.127) (type solid)) (layer "F.SilkS"))
-    (fp_arc (start 10.541 6.985) (mid 9.983038 8.332038) (end 8.636 8.89)
-      (stroke (width 0.127) (type solid)) (layer "F.SilkS"))
-    (fp_arc (start 11.551272 -4.491272) (mid 11.904644 -4.344724) (end 12.051 -3.991272)
-      (stroke (width 0.127) (type default)) (layer "F.SilkS"))
-    (fp_arc (start 12.051 4.004) (mid 11.904553 4.357553) (end 11.551 4.504)
-      (stroke (width 0.127) (type default)) (layer "F.SilkS"))
     (fp_circle (center 9.42 -7.807) (end 9.674 -7.807)
       (stroke (width 0.5) (type solid)) (fill solid) (layer "F.SilkS"))
@@
     (fp_rect (start -10.425 -8.9) (end 10.55 8.9)
       (stroke (width 0.05) (type default)) (fill none) (layer "F.CrtYd"))
+    (fp_line (start -8.509 -8.89) (end 8.636 -8.89)
+      (stroke (width 0.127) (type solid)) (layer "F.Fab"))
+    (fp_line (start -8.509 8.89) (end 8.636 8.89)
+      (stroke (width 0.127) (type solid)) (layer "F.Fab"))
+    (fp_line (start 10.541 -4.495) (end 11.551272 -4.491272)
+      (stroke (width 0.127) (type solid)) (layer "F.Fab"))
+    (fp_line (start 10.541 6.985) (end 10.541 -6.985)
+      (stroke (width 0.1) (type solid)) (layer "F.Fab"))
+    (fp_line (start 10.541 6.985) (end 10.541 -6.985)
+      (stroke (width 0.127) (type solid)) (layer "F.Fab"))
+    (fp_line (start 11.551 4.504) (end 10.541 4.504)
+      (stroke (width 0.127) (type solid)) (layer "F.Fab"))
+    (fp_line (start 12.051 -3.991272) (end 12.051 4.004)
+      (stroke (width 0.127) (type solid)) (layer "F.Fab"))
     (fp_rect (start -10.425 -8.9) (end 10.55 8.9)
       (stroke (width 0.1) (type default)) (fill none) (layer "F.Fab"))
+    (fp_arc (start 8.636 -8.89) (mid 9.983038 -8.332038) (end 10.541 -6.985)
+      (stroke (width 0.127) (type solid)) (layer "F.Fab"))
+    (fp_arc (start 10.541 6.985) (mid 9.983038 8.332038) (end 8.636 8.89)
+      (stroke (width 0.127) (type solid)) (layer "F.Fab"))
+    (fp_arc (start 11.551272 -4.491272) (mid 11.904644 -4.344724) (end 12.051 -3.991272)
+      (stroke (width 0.127) (type default)) (layer "F.Fab"))
+    (fp_arc (start 12.051 4.004) (mid 11.904553 4.357553) (end 11.551 4.504)
+      (stroke (width 0.127) (type default)) (layer "F.Fab"))
     (fp_circle (center 9.426 -7.804) (end 9.68 -7.804)
       (stroke (width 0.5) (type solid)) (fill solid) (layer "F.Fab"))
