File: pcb/RishiStarbie.kicad_sch (KiCad schematic)
At the start: 7 parts, among them J1 OLED, J2 MPU6050, SW1 MX switch, SW2 MX switch, U1 XIAO-ESP32-C3, U2 DHT11

Commit message: Move off-board XIAO silkscreen to fab layer, rename footprint to XIAO-ESP32-C3-DIP
Parts:
- U1: footprint Imported Parts:XIAO-ESP32-C6-DIP -> Imported Parts:XIAO-ESP32-C3-DIP
Changed lines of the file:
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@@
         (font
           (size 1.27 1.27))))
-    (property "Footprint" "Imported Parts:XIAO-ESP32-C6-DIP"
+    (property "Footprint" "Imported Parts:XIAO-ESP32-C3-DIP"
       (at 228.6 69.85 0)
       (effects
